File: Ares_FC/Ares_FC.kicad_sch (KiCad schematic)
At the start: 2 parts, among them IC1 STM32H742VIT6, J1 MICRO-SD-CARD

Commit message: .
Parts:
- removed IC1: STM32H742VIT6, STM32H742VIT6:QFP50P1600X1600X160-100N, symbol STM32H742VIT6:STM32H742VIT6
- removed J1: MICRO-SD-CARD, MICRO-SD-CARD:MICROSDCARD, symbol MICRO-SD-CARD:MICRO-SD-CARD
- added BigAssLPFCapacitor1: 220u, symbol Device:C_Polarized
- added Boot0_Button1, Boot0_Button2, GP_PushButton1, SW1: SW_Push, symbol Switch:SW_Push
- added C1: 1u, symbol Device:C
- added C2, C3, C4, C5, C6, C7: 100n, symbol Device:C
- added CL1, CL2: 10p, symbol Device:C
- added GP_Poti1, GP_Poti2, Speed_Poti1: 0-200k, symbol Device:R_Trim
- added IC1: STM32F411RET6, QFP50P1200X1200X160-64N, symbol STM32F411RET6:STM32F411RET6
- added L1: L, symbol Device:L
- added R1, R2: 0, symbol Device:R
- added R3, R4: 10k, symbol Device:R
- added R5: 22k, symbol Device:R
- added R6, R7, R9: 220k, symbol Device:R
- added R8: n.p., symbol Device:R
- added U2: ~, symbol JST_Connectors:JST-PH2.0mm
- added U3: ~, symbol JST_Connectors:JST-PH_2mm_6Pin
- added Y1: 830107871909, 830107871909, symbol 830107871909:830107871909
Connections:
- new net: CL1.1, R1.1, Y1.1 (CRYSTAL_1)
- new net: CL2.1, R2.2, Y1.3 (CRYSTAL_2)
- new net: R8.1, U3.1
- new net ADC_0: GP_Poti1.2, IC1.14 (PA0), R7.1
- new net ADC_1: GP_Poti2.2, IC1.15 (PA1), R9.1
- new net ADC_10: IC1.8 (PC0)
- new net ADC_11: IC1.9 (PC1)
- new net ADC_12: IC1.10 (PC2)
- new net ADC_13: IC1.11 (PC3)
- new net ADC_14: IC1.24 (PC4)
- new net ADC_15: IC1.25 (PC5)
- new net ADC_2: IC1.16 (PA2)
- new net ADC_3: IC1.17 (PA3)
- new net ADC_4: IC1.20 (PA4)
- new net ADC_5: IC1.21 (PA5)
- new net ADC_6: IC1.22 (PA6)
- new net ADC_7: IC1.23 (PA7)
- new net ADC_8: GP_PushButton1.1, IC1.26 (PB0), R5.1
- new net ADC_9: IC1.27 (PB1), R6.1, Speed_Poti1.2
- new net BOOT0: Boot0_Button1.1, IC1.60 (BOOT0), R3.1
- new net BOOT1: Boot0_Button2.1, IC1.28 (PB2), R4.1
- new net GND: BigAssLPFCapacitor1.2, C1.2, C2.2, C3.2, C4.2, C5.2, C6.2, C7.2, CL1.2, CL2.2, IC1.12 (VSSA/VREF-), IC1.18 (VSS_1), IC1.31 (VSS_2), IC1.47 (VSS_3), IC1.63 (VSS_4), R3.2, R4.2, R5.2, R6.2, R7.2, R9.2, SW1.1, U2.2 (V-), U3.3, Y1.2 (GND_1), Y1.4 (GND_2)
- new net NRST: C2.1, IC1.7 (NRST), SW1.2, U3.5
- new net OSC_IN: IC1.5 (PH0-OSC_IN), R1.2
- new net OSC_OUT: IC1.6 (PH1-OSC_OUT), R2.1
- new net SWD-CLK: IC1.49 (PA14), U3.2
- new net SWD-I/O: IC1.46 (PA13), U3.4
- new net SWD-TRACESWO: IC1.55 (PB3), U3.6
- new net VDD: BigAssLPFCapacitor1.1, Boot0_Button1.2, Boot0_Button2.2, C3.1, C4.1, C5.1, C6.1, C7.1, GP_Poti1.1, GP_Poti2.1, GP_PushButton1.2, IC1.1 (VBAT), IC1.19 (VDD_1), IC1.32 (VDD_2), IC1.48 (VDD_3), IC1.64 (VDD_4), L1.2, R8.2, Speed_Poti1.1, U2.1 (V+)
- new net VDDF: C1.1, IC1.13 (VDDA/VREF+), L1.1
Other:
- note added: "1 x 100nF Cap für jeden VDD-Eingang. Direkt davor platziert."
- note added: "General Purpose Push Button"
- note added: "Poti zur Geschwindigkeitseinstellung und 2 Potis für die PI-Regelung"
- note added: "Power Connection to Power Board via JST PH 2.0mm Connector"
- note added: "SWD für Debugging und Flashing nutzen!!"
- note added: "ToDos: - UART, I2C und SPI Connector implementieren - UART Verbindung via USB-UART Bridge realisieren (Zur Seriellen Ausgabe an PC)"
