File: Beestaeuber_v1/Beestaeuber_v1_project/Beestaeuber_v1_project.kicad_sch (KiCad schematic)
At the start: 74 parts, among them IC1 AT7456E, IC2 DPS368XTSA1, IC3 USBLC6-2SC6, IC4 STM32H753VIT6, IC5 MP2315SGJ-Z, J10 PWM Connector 4, J11 PWM Connector 4, J12 PWM Connector 3, J13 PWM Connector 3, J14 GSB1C41110SSHR, J16 Conn_02x05_Top_Bottom_Mountin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, J17 MEM2061-01-188-00-A, J2 ELRS_Receiver, J4 PWM Connector 1, J5 PWM Connector 2, J6 CAM Connector, J7 VTX Output, J8 PWM Connector 1, J9 PWM Connector 2, U2 ICM-40609-D, U3 LD1117S33TR

Commit message: .
Parts:
- added C26, C30, C31: 22u, Capacitor_SMD:C_0603_1608Metric, symbol Device:C
- added C27, C28, C29, C32, C33, C34: 100n, Capacitor_SMD:C_0603_1608Metric, symbol Device:C
- added J1: WS2812_1, symbol Connector:Conn_01x03_Pin
- added J15: WS2812_3, symbol Connector:Conn_01x03_Pin
- added J18: WS2812_4, symbol Connector:Conn_01x03_Pin
- added J19: GPS, Connector_JST:JST_XH_B4B-XH-AM_1x04_P2.50mm_Vertical, symbol JST_XH_4Pin_female:B4B-XH-AM__LF__SN_
- added J3: WS2812_2, symbol Connector:Conn_01x03_Pin
- added L1: 4u2, symbol Device:L
- added R29: 33k, symbol Device:R
- added R30: 40k2, symbol Device:R
- added R31: 12k7, symbol Device:R
- added R32: 100k, symbol Device:R
- added R33: 7k5, symbol Device:R
- added R34: 10, symbol Device:R
- added R35: 499k, symbol Device:R
- added R36, R37, R38, R39: x, symbol Device:R
- added R7: 0, symbol Device:R
- added U1, U4: APA102C, APA102C:SON160P500X500X140-6N, symbol WS2812_APA102C:APA102C
- C8, C9, IC1, J6, J7, U3: now not fitted
- J2: value ELRS_Receiver -> ELRS
Connections:
- net +3V3: now also C29.1, C30.1, C31.1, L1.2, R30.1
- net +5V: now also IC5.2 (IN), C26.1, C32.1, C33.1, C34.1, J1.3 (Pin_3), J15.3 (Pin_3), J18.3 (Pin_3), J3.3 (Pin_3), R35.1, R37.1, R38.1, U1.4 (VCC), U4.4 (VCC)
- net GND: now also IC5.4 (GND), C26.2, C27.2, C30.2, C31.2, C32.2, C33.2, C34.2, J1.1 (Pin_1), J15.1 (Pin_1), J18.1 (Pin_1), J3.1 (Pin_1), R31.2, R33.2, R36.2, R39.2, U1.3 (GND), U4.3 (GND)
- net VBUS: now also R7.1
- net USB_VBUS: now reaches IC4.68 (PA9)
- net USB_VBUS: now also R7.2
- net MP2315S_AAM: now reaches IC5.1 (AAM)
- net MP2315S_AAM: now also R32.2, R33.1
- net MP2315S_SW: now reaches IC5.3 (SW)
- net MP2315S_SW: now also C28.1, L1.1
- net at IC5.5 (BST): now also R34.2
- net at IC5.6 (EN): now also R35.2
- net MP2315S_VCC: now reaches IC5.7 (VCC)
- net MP2315S_VCC: now also C27.1, R32.1
- net at IC5.8 (FB): now also R29.2
- new net: R38.2, R39.1, U4.6 (DO)
- new net: R36.1, R37.2, U4.5 (CO)
- new net: C29.2, R29.1, R30.2, R31.1
- new net: U1.6 (DO), U4.1 (DI)
- new net: U1.5 (CO), U4.2 (CI)
- new net: C28.2, R34.1
- new net APA102C_ClockIn: U1.2 (CI)
- new net APA102C_DataIn: U1.1 (DI)
- new net WS2812_1_Data: J1.2 (Pin_2)
- new net WS2812_2_Data: J3.2 (Pin_2)
- new net WS2812_3_Data: J15.2 (Pin_2)
- new net WS2812_4_Data: J18.2 (Pin_2)
Other:
- note added: "> 1206 oder 1210 SMD Part (>0.25Watts)"
- note added: "Backup LDO Space"
- note added: "Might need Adjustments (lower than 500k)"
- note added: "Power"
- note added: "SD Card"
- note added: "Sets VOut to 3.3V"
- note added: "ToDo: -Interrupt Pins verbinden -Buzzer Output Pad -Add 25MHz HSE Oscillator for MCU -Cam Input and VTX Output + Chip Integration -Choose SMD JST Connectors -Add Magnetometer and other Sensors -GPS -Cam Input -VTX Output -5V Input/Output Pads -Analog Input/Output Pads -PWM Outputs for Servos -Battery Input Pad for measuring Voltage -Add Level Shifters for ELRS and GPS Connection"
- note added: "USB-C"
- note removed: "-GPS -Barometer -Cam Input -VTX Output -SD Card Slot -8 PWM Outputs -5V Input/Output Pads -Analog Input/Output Pads -PWM Outputs for Servos -Battery Input Pad for measuring Voltage"
- note removed: "4 x WS2812 Outputs 1 x On-board WS2812 LED"
- note removed: "ELRS"
- note removed: "ToDo: -Add ESPC6 for Bluetooth Connectifity -Add USB-C PD Controller for more Power -Interrupt Pins verbinden"
- note removed: "ersetzen durch switching regulator -> efficiency"
- moved on the sheet: C10, C11, C12, C13, C14, C15, C16, C17, C18, C19, C2, C20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
